File: flatsat-main.kicad_pcb (KiCad board)
At the start: 4 copper layers, 120 x 150 mm, 26 parts, among them P1 OBC_PGM, P2 PAY_PGM, P3 COM_PGM, P4 PGM_ALL, P5 EPS_PGM, SW1 RST_OBC, SW2 RST_PAY, SW3 RST_COM, SW4 RST_EPS

Commit message: done
wohoo
Parts:
- moved DBG1 21.8 mm to (151.8, 143.3), turned to 270 degrees
- moved G1 4.49 mm to (104.2, 41.5)
- moved G2 4.49 mm to (104.2, 106.9)
- turned D1 to 180 degrees
- turned D4 to 180 degrees
- renumbered P4 to ALL, P3 to COM, SW3 to COM, P5 to EPS, SW4 to EPS, P1 to OBC, SW1 to OBC, P2 to PAY, SW2 to PAY
Routing:
- net /OBC_SCK_A: track 0.00 -> 198.5 mm, vias 0 -> 3
- net /SCK_A_COMMON: track 0.00 -> 193.1 mm, vias 0 -> 2
- net /OBC_MOSI_A: track 0.00 -> 188.1 mm, vias 0 -> 1
- net /OBC_RST: track 0.00 -> 187.6 mm, vias 0 -> 1
- net /MOSI_A_COMMON: track 0.00 -> 186.5 mm, vias 0 -> 2
- net /COM_RST: track 0.00 -> 175.9 mm, vias 0 -> 2
- net /PAY_RST: track 0.00 -> 175.0 mm, vias 0 -> 2
- net /EPS_SCK_A: track 0.00 -> 161.5 mm, vias 0 -> 1
- net /EPS_MOSI_A: track 0.00 -> 161.0 mm, vias 0 -> 1
- net /MISO_A_COMMON: track 0.00 -> 137.7 mm
- net /CANH: track 0.00 -> 129.3 mm
- net /OBC_MISO_A: track 0.00 -> 128.7 mm
- net /VIN: track 0.00 -> 124.8 mm
- net /EPS_RST: track 0.00 -> 123.0 mm, vias 0 -> 1
- net /EPS_MISO_A: track 0.00 -> 121.7 mm
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- added copper zone on VCC, net /3V3CRIT
- added copper zone on GND, net GND
Other:
- board text added: "3V3"
- board text added: "CANH"
- board text added: "CANL"
- board text added: "GND"
- board text added: "RX"
- board text added: "TX ALL"
- board text added: "TX COM"
- board text added: "TX EPS"
- board text added: "TX OBC"
- board text added: "TX PAY"
- board text added: "VIN"
